File: AutoHuerta_Kicad/hidroponia.kicad_sch (KiCad schematic)
At the start: 37 parts, among them J1 bornera, J2 bornera, J3 Barrel_Jack, J4 pin, J6 Pin, J7 Pin, K1 RELAY, Q1 BC817, Q2 BS170F, Q3 BC817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

Commit message: PCB
cambios en el pcb
Parts:
- U2, U4, U6: footprint Package_SO:SSO-4_6.7x5.1mm_P2.54mm_Clearance8mm -> Package_DIP:DIP-4_W7.62mm_LongPads
Connections:
- net +12V: now also J7.6 (Pin_6); no longer J7.2 (Pin_2)
- net +5V: now also J7.2 (Pin_2); no longer J7.6 (Pin_6)
- net BOMBA: now also U1.27 (A2); no longer U1.26 (A1)
- net VEL: now also J6.1 (Pin_1), U1.26 (A1); no longer J6.2 (Pin_2), U1.27 (A2)
- net at D5.1 (K), D6.2 (A), Q3.3 (C): now also J6.2 (Pin_2); no longer J6.1 (Pin_1)
Changed lines of the file:
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@@
 	(wire
 		(pts
-			(xy 232.41 100.33) (xy 220.98 100.33)
-		)
-		(stroke
-			(width 0)
-			(type default)
-		)
-	)
-	(wire
-		(pts
 			(xy 185.42 105.41) (xy 186.69 105.41)
 		)
@@
 		)
 	)
+	(wire
+		(pts
+			(xy 163.83 143.51) (xy 163.83 144.78)
+		)
+		(stroke
+			(width 0)
+			(type default)
+		)
+	)
 	(bus
 		(pts
@@
 	(wire
 		(pts
-			(xy 153.67 143.51) (xy 153.67 144.78)
+			(xy 212.09 120.65) (xy 220.98 120.65)
 		)
 		(stroke
@@
 	(wire
 		(pts
-			(xy 232.41 93.98) (xy 232.41 100.33)
+			(xy 30.48 99.06) (xy 33.02 99.06)
 		)
 		(stroke
@@
 	(wire
 		(pts
-			(xy 212.09 120.65) (xy 220.98 120.65)
+			(xy 33.02 137.16) (xy 31.75 137.16)
 		)
 		(stroke
@@
 		)
 	)
-	(wire
+	(bus
 		(pts
-			(xy 30.48 99.06) (xy 33.02 99.06)
+			(xy 26.67 92.71) (xy 26.67 114.3)
 		)
 		(stroke
@@
 	(wire
 		(pts
-			(xy 33.02 137.16) (xy 31.75 137.16)
-		)
-		(stroke
-			(width 0)
-			(type default)
-		)
-	)
-	(bus
-		(pts
-			(xy 26.67 92.71) (xy 26.67 114.3)
+			(xy 232.41 88.9) (xy 232.41 82.55)
 		)
 		(stroke
@@
 	(wire
 		(pts
-			(xy 232.41 82.55) (xy 220.98 82.55)
+			(xy 220.98 82.55) (xy 232.41 82.55)
 		)
 		(stroke
@@
 		)
 	)
-	(wire
-		(pts
-			(xy 50.8 58.42) (xy 52.07 58.42)
-		)
-		(stroke
-			(width 0)
-			(type default)
-		)
-	)
 	(bus
 		(pts
@@
 	(wire
 		(pts
-			(xy 50.8 53.34) (xy 52.07 53.34)
+			(xy 50.8 55.88) (xy 52.07 55.88)
 		)
 		(stroke
@@
 	(wire
 		(pts
+			(xy 229.87 93.98) (xy 232.41 93.98)
+		)
+		(stroke
+			(width 0)
+			(type default)
+		)
+	)
+	(wire
+		(pts
 			(xy 119.38 25.4) (xy 125.73 25.4)
 		)
@@
 	(wire
 		(pts
+			(xy 231.14 100.33) (xy 220.98 100.33)
+		)
+		(stroke
+			(width 0)
+			(type default)
+		)
+	)
+	(wire
+		(pts
 			(xy 15.24 62.23) (xy 15.24 60.96)
 		)
@@
 	(wire
 		(pts
+			(xy 50.8 53.34) (xy 52.07 53.34)
+		)
+		(stroke
+			(width 0)
+			(type default)
+		)
+	)
+	(wire
+		(pts
 			(xy 132.08 30.48) (xy 132.08 25.4)
 		)
@@
 	(wire
 		(pts
+			(xy 50.8 58.42) (xy 52.07 58.42)
+		)
+		(stroke
+			(width 0)
+			(type default)
+		)
+	)
+	(wire
+		(pts
 			(xy 106.68 53.34) (xy 107.95 53.34)
 		)
@@
 		)
 	)
-	(wire
-		(pts
-			(xy 232.41 82.55) (xy 232.41 88.9)
-		)
-		(stroke
-			(width 0)
-			(type default)
-		)
-	)
 	(bus
 		(pts
@@
 	(wire
 		(pts
-			(xy 231.14 91.44) (xy 232.41 91.44)
-		)
-		(stroke
-			(width 0)
-			(type default)
-		)
-	)
-	(wire
-		(pts
 			(xy 30.48 97.79) (xy 30.48 99.06)
 		)
@@
 	(wire
 		(pts
-			(xy 50.8 55.88) (xy 52.07 55.88)
-		)
-		(stroke
-			(width 0)
-			(type default)
-		)
-	)
-	(wire
-		(pts
 			(xy 220.98 81.28) (xy 220.98 82.55)
 		)
@@
 	(wire
 		(pts
+			(xy 232.41 91.44) (xy 231.14 91.44)
+		)
+		(stroke
+			(width 0)
+			(type default)
+		)
+	)
+	(wire
+		(pts
 			(xy 166.37 143.51) (xy 166.37 144.78)
 		)
@@
 	(wire
 		(pts
+			(xy 153.67 143.51) (xy 153.67 144.78)
+		)
+		(stroke
+			(width 0)
+			(type default)
+		)
+	)
+	(wire
+		(pts
 			(xy 22.86 66.04) (xy 19.05 66.04)
 		)
@@
 	(wire
 		(pts
-			(xy 163.83 143.51) (xy 163.83 144.78)
+			(xy 231.14 91.44) (xy 231.14 100.33)
 		)
 		(stroke
@@
 	(global_label "BOMBA"
 		(shape input)
-		(at 52.07 55.88 0)
+		(at 52.07 53.34 0)
 		(fields_autoplaced yes)
 		(effects
@@
 		)
 		(property "Intersheetrefs" "${INTERSHEET_REFS}"
-			(at 61.4657 55.88 0)
+			(at 61.4657 53.34 0)
 			(effects
 				(font
@@
 	(global_label "VEL"
 		(shape input)
-		(at 231.14 91.44 180)
+		(at 229.87 93.98 180)
 		(fields_autoplaced yes)
 		(effects
@@
 		)
 		(property "Intersheetrefs" "${INTERSHEET_REFS}"
-			(at 224.8891 91.44 0)
+			(at 223.6191 93.98 0)
 			(effects
 				(font
@@
 	(global_label "VEL"
 		(shape input)
-		(at 52.07 53.34 0)
+		(at 52.07 55.88 0)
 		(fields_autoplaced yes)
 		(effects
@@
 		)
 		(property "Intersheetrefs" "${INTERSHEET_REFS}"
-			(at 58.3209 53.34 0)
+			(at 58.3209 55.88 0)
 			(effects
 				(font
@@
 			)
 		)
-		(property "Footprint" "Package_SO:SSO-4_6.7x5.1mm_P2.54mm_Clearance8mm"
+		(property "Footprint" "Package_DIP:DIP-4_W7.62mm_LongPads"
 			(at 96.52 113.03 0)
 			(effects
@@
 			)
 		)
-		(property "Footprint" "Package_SO:SSO-4_6.7x5.1mm_P2.54mm_Clearance8mm"
+		(property "Footprint" "Package_DIP:DIP-4_W7.62mm_LongPads"
 			(at 93.98 55.88 0)
 			(effects
@@
 	(symbol
 		(lib_id "power:+12V")
-		(at 153.67 143.51 0)
+		(at 163.83 143.51 0)
 		(unit 1)
 		(exclude_from_sim no)
@@
 		(dnp no)
 		(property "Reference" "#PWR027"
-			(at 153.67 147.32 0)
+			(at 163.83 147.32 0)
 			(effects
 				(font
@@
 		)
 		(property "Value" "+12V"
-			(at 153.416 137.16 0)
+			(at 163.576 137.16 0)
 			(effects
 				(font
@@
 		)
 		(property "Footprint" ""
-			(at 153.67 143.51 0)
+			(at 163.83 143.51 0)
 			(effects
 				(font
@@
 		)
 		(property "Datasheet" ""
-			(at 153.67 143.51 0)
+			(at 163.83 143.51 0)
 			(effects
 				(font
@@
 		)
 		(property "Description" "Power symbol creates a global label with name \"+12V\""
-			(at 153.67 143.51 0)
+			(at 163.83 143.51 0)
 			(effects
 				(font
@@
 	(symbol
 		(lib_id "power:+5V")
-		(at 163.83 143.51 0)
+		(at 153.67 143.51 0)
 		(unit 1)
 		(exclude_from_sim no)
@@
 		(dnp no)
 		(property "Reference" "#PWR028"
-			(at 163.83 147.32 0)
+			(at 153.67 147.32 0)
 			(effects
 				(font
@@
 		)
 		(property "Value" "+5V"
-			(at 163.83 138.43 0)
+			(at 153.67 137.414 0)
 			(effects
 				(font
@@
 		)
 		(property "Footprint" ""
-			(at 163.83 143.51 0)
+			(at 153.67 143.51 0)
 			(effects
 				(font
@@
 		)
 		(property "Datasheet" ""
-			(at 163.83 143.51 0)
+			(at 153.67 143.51 0)
 			(effects
 				(font
@@
 		)
 		(property "Description" "Power symbol creates a global label with name \"+5V\""
-			(at 163.83 143.51 0)
+			(at 153.67 143.51 0)
 			(effects
 				(font
@@
 			)
 		)
-		(property "Footprint" "Package_SO:SSO-4_6.7x5.1mm_P2.54mm_Clearance8mm"
+		(property "Footprint" "Package_DIP:DIP-4_W7.62mm_LongPads"
 			(at 189.23 113.03 0)
 			(effects

Commit message: actualizacion de PCB
pruebas
Connections:
- net +5V: now also J7.4 (Pin_4); no longer J7.2 (Pin_2)
- net GND: now also J7.2 (Pin_2); no longer J7.4 (Pin_4)
Changed lines of the file:
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@@
 	(wire
 		(pts
+			(xy 153.67 143.51) (xy 153.67 144.78)
+		)
+		(stroke
+			(width 0)
+			(type default)
+		)
+	)
+	(wire
+		(pts
 			(xy 119.38 110.49) (xy 120.65 110.49)
 		)
@@
 	(wire
 		(pts
-			(xy 158.75 143.51) (xy 158.75 144.78)
-		)
-		(stroke
-			(width 0)
-			(type default)
-		)
-	)
-	(wire
-		(pts
 			(xy 50.8 50.8) (xy 52.07 50.8)
 		)
@@
 	(wire
 		(pts
-			(xy 166.37 143.51) (xy 166.37 144.78)
+			(xy 158.75 143.51) (xy 158.75 144.78)
 		)
 		(stroke
@@
 	(wire
 		(pts
-			(xy 153.67 143.51) (xy 153.67 144.78)
+			(xy 166.37 143.51) (xy 166.37 144.78)
 		)
 		(stroke
@@
 	(symbol
 		(lib_id "power:+5V")
-		(at 153.67 143.51 0)
+		(at 158.75 143.51 0)
 		(unit 1)
 		(exclude_from_sim no)
@@
 		(dnp no)
 		(property "Reference" "#PWR028"
-			(at 153.67 147.32 0)
+			(at 158.75 147.32 0)
 			(effects
 				(font
@@
 		)
 		(property "Value" "+5V"
-			(at 153.67 137.414 0)
+			(at 158.75 137.414 0)
 			(effects
 				(font
@@
 		)
 		(property "Footprint" ""
-			(at 153.67 143.51 0)
+			(at 158.75 143.51 0)
 			(effects
 				(font
@@
 		)
 		(property "Datasheet" ""
-			(at 153.67 143.51 0)
+			(at 158.75 143.51 0)
 			(effects
 				(font
@@
 		)
 		(property "Description" "Power symbol creates a global label with name \"+5V\""
-			(at 153.67 143.51 0)
+			(at 158.75 143.51 0)
 			(effects
 				(font
@@
 	(symbol
 		(lib_id "power:GND")
-		(at 158.75 143.51 180)
+		(at 153.67 143.51 180)
 		(unit 1)
 		(exclude_from_sim no)
@@
 		(dnp no)
 		(property "Reference" "#PWR029"
-			(at 158.75 137.16 0)
+			(at 153.67 137.16 0)
 			(effects
 				(font
@@
 		)
 		(property "Value" "GND"
-			(at 158.242 139.954 0)
+			(at 153.162 139.954 0)
 			(effects
 				(font
@@
 		)
 		(property "Footprint" ""
-			(at 158.75 143.51 0)
+			(at 153.67 143.51 0)
 			(effects
 				(font
@@
 		)
 		(property "Datasheet" ""
-			(at 158.75 143.51 0)
+			(at 153.67 143.51 0)
 			(effects
 				(font
@@
 		)
 		(property "Description" "Power symbol creates a global label with name \"GND\" , ground"
-			(at 158.75 143.51 0)
+			(at 153.67 143.51 0)
 			(effects
 				(font
